File: pcb/stm_audio_board_V2/_autosave-stm_audio_board_V2.kicad_pcb (KiCad board)
At the start: 4 copper layers, 113 parts, among them J1 Power conn, J2 STlink, J3 Audio_sig, J4 Conn_01x10_pots_internal, J5 SPI, J6 Conn_01x03_pot_ext, J7 GuitarIN, J8 GuitarOUT_R, J9 GuitarOUT_L, SW1 SW_SPST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

Commit message: Schematic divided into pages, Global connectors added
Connections:
- C54 pad 1: /filters/pot5 -> POT5
- C55 pad 1: /filters/pot1 -> POT1
- C56 pad 1: /filters/pot6 -> POT6
- C57 pad 1: /filters/pot2 -> POT2
- C58 pad 1: /filters/pot7 -> POT7
- C59 pad 1: /filters/pot3 -> POT3
- C60 pad 1: /filters/pot8 -> POT8
- C61 pad 1: /filters/pot_external -> POT_EXT
- C62 pad 1: /filters/pot4 -> POT4
- U1 pad 15: /MCU/pot1 -> POT1
- U1 pad 16: /MCU/pot2 -> POT2
- U1 pad 17: /MCU/pot3 -> POT3
- U1 pad 18: /MCU/pot4 -> POT4
- U1 pad 32: /MCU/pot5 -> POT5
- U1 pad 33: /MCU/pot6 -> POT6
- U1 pad 63: /MCU/pot7 -> POT7
- U1 pad 64: /MCU/pot8 -> POT8
- U1 pad 65: /MCU/pot_external -> POT_EXT
