File: pcb/stm_audio_board_V2/Input_stage.kicad_sch (KiCad schematic)
At the start: 19 parts, among them J7 GuitarIN, U3 AD1974, U4 OP275

Commit message: added choke to analog pwr, created 5 V rail, decided to pivot and use codec instead dedicated hardware
Parts:
- added C18 (x2): 12p, Capacitor_SMD:C_0603_1608Metric_Pad1.08x0.95mm_HandSolder, symbol Device:C_Small
- added R4: 1Meg, Resistor_SMD:R_0805_2012Metric_Pad1.20x1.40mm_HandSolder, symbol Device:R
- added Y1: Crystal_GND24, Crystal:Crystal_SMD_5032-4Pin_5.0x3.2mm, symbol Device:Crystal_GND24
- R8, R9: value 237R -> 240R
Connections:
- net AUDIO_IN: now also R4.1
- net GND: now also C18.1, C18.2, Y1.2, Y1.4
- net GNDA: now also R4.2; no longer U4.3 (+)
- net at U3.2 (MCLKI/XI): now also C18.1, Y1.3
- net at U3.3 (MCLKO/XO): now also C18.2, Y1.1
- net at C17.1, R5.2, U4.2 (-): no longer R4.1
- new net: R4.1, U4.3 (+)
Other:
- moved on the sheet: C18, J7, R4
