File: pcb/stm_audio_board_V2/_autosave-Power.kicad_sch (KiCad schematic)
At the start: 42 parts, among them U10 TL072, U2 AMS1117-3.3, U4 OP275, U5 AMS1117-3.3, U7 OP275, U8 AMS1117-5.0, U9 L7809

Commit message: Update #auto_saved_files#, Power.kicad_sch, and 6 more files...
Other:
- note added: "CODEC power connecntions"
Changed lines of the file:
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@@
     (stroke (width 0) (type default))
+  )
+  (rectangle (start 15.24 180.34) (end 116.84 232.41)
+    (stroke (width 0) (type default))
+    (fill (type none))
   )
   (rectangle (start 129.54 20.32) (end 233.68 67.31)
@@
     (effects (font (size 1.27 1.27)) (justify left bottom))
   )
+  (text "CODEC power connecntions\n" (at 15.24 179.07 0)
+    (effects (font (size 1.27 1.27)) (justify left bottom))
+  )
