File: pcb/stm_audio_board_V2/Power.kicad_sch (KiCad schematic)
At the start: 28 parts, among them U2 OP275, U4 OP275, U5 AMS1117-3.3, U8 L78M09CDT, U9 LF33_TO252

Commit message: Update #auto_saved_files#, Connectors.kicad_sch, and 18 more files...
Parts:
- removed D4: 1N4148, Diode_THT:D_DO-35_SOD27_P7.62mm_Horizontal, symbol Diode:1N4148
- C28, C29: footprint Capacitor_THT:CP_Radial_D6.3mm_P2.50mm -> Capacitor_SMD:CP_Elec_6.3x7.7
- C4: footprint Capacitor_SMD:CP_Elec_6.3x7.7 -> Capacitor_SMD:C_1206_3216Metric_Pad1.33x1.80mm_HandSolder
Changed lines of the file:
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@@
   (junction (at 168.91 198.12) (diameter 0) (color 0 0 0 0)
   )
-  (junction (at 171.45 138.43) (diameter 0) (color 0 0 0 0)
-  )
   (junction (at 165.1 138.43) (diameter 0) (color 0 0 0 0)
   )
@@
   (junction (at 228.6 92.71) (diameter 0) (color 0 0 0 0)
   )
-  (junction (at 195.58 138.43) (diameter 0) (color 0 0 0 0)
-  )
   (junction (at 158.75 39.37) (diameter 0) (color 0 0 0 0)
   )
@@
     (stroke (width 0) (type default))
   )
-  (wire (pts (xy 171.45 138.43) (xy 175.26 138.43))
-    (stroke (width 0) (type default))
-  )
   (wire (pts (xy 171.45 218.44) (xy 168.91 218.44))
     (stroke (width 0) (type default))
@@
     (stroke (width 0) (type default))
   )
-  (wire (pts (xy 182.88 128.27) (xy 171.45 128.27))
-    (stroke (width 0) (type default))
-  )
   (wire (pts (xy 208.28 83.82) (xy 209.55 83.82))
     (stroke (width 0) (type default))
@@
     (stroke (width 0) (type default))
   )
-  (wire (pts (xy 165.1 138.43) (xy 171.45 138.43))
+  (wire (pts (xy 165.1 138.43) (xy 175.26 138.43))
     (stroke (width 0) (type default))
   )
@@
     (stroke (width 0) (type default))
   )
-  (wire (pts (xy 195.58 128.27) (xy 195.58 138.43))
-    (stroke (width 0) (type default))
-  )
   (wire (pts (xy 199.39 213.36) (xy 201.93 213.36))
     (stroke (width 0) (type default))
@@
     (stroke (width 0) (type default))
   )
-  (wire (pts (xy 195.58 138.43) (xy 198.12 138.43))
+  (wire (pts (xy 193.04 138.43) (xy 198.12 138.43))
     (stroke (width 0) (type default))
   )
@@
     (stroke (width 0) (type default))
   )
-  (wire (pts (xy 193.04 138.43) (xy 195.58 138.43))
-    (stroke (width 0) (type default))
-  )
   (wire (pts (xy 109.22 36.83) (xy 109.22 39.37))
     (stroke (width 0) (type default))
@@
     (stroke (width 0) (type default))
   )
-  (wire (pts (xy 190.5 128.27) (xy 195.58 128.27))
-    (stroke (width 0) (type default))
-  )
   (wire (pts (xy 201.93 205.74) (xy 201.93 208.28))
     (stroke (width 0) (type default))
@@
   )
   (wire (pts (xy 199.39 205.74) (xy 201.93 205.74))
-    (stroke (width 0) (type default))
-  )
-  (wire (pts (xy 171.45 128.27) (xy 171.45 138.43))
     (stroke (width 0) (type default))
   )
@@
       (effects (font (size 1.27 1.27)) (justify left))
     )
-    (property "Footprint" "Capacitor_SMD:CP_Elec_6.3x7.7" (at 170.18 46.99 0)
+    (property "Footprint" "Capacitor_SMD:C_1206_3216Metric_Pad1.33x1.80mm_HandSolder" (at 170.18 46.99 0)
       (effects (font (size 1.27 1.27)) hide)
     )
@@
       (effects (font (size 1.27 1.27)) (justify left))
     )
-    (property "Footprint" "Capacitor_THT:CP_Radial_D6.3mm_P2.50mm" (at 175.26 147.32 0)
+    (property "Footprint" "Capacitor_SMD:CP_Elec_6.3x7.7" (at 175.26 147.32 0)
       (effects (font (size 1.27 1.27)) hide)
     )
@@
         (path "/6997cf63-2615-4e49-9471-e7da1b6bae71/2eb2ee8f-ab98-4666-97f0-bfacb073bc88"
           (reference "#PWR061") (unit 1)
-        )
-      )
-    )
-  )
-  (symbol (lib_id "Diode:1N4148") (at 186.69 128.27 0) (unit 1)
-    (in_bom yes) (on_board yes) (dnp no)
-    (property "Reference" "D4" (at 186.69 123.19 0)
-      (effects (font (size 1.27 1.27)))
-    )
-    (property "Value" "1N4148" (at 186.69 125.73 0)
-      (effects (font (size 1.27 1.27)))
-    )
-    (property "Footprint" "Diode_THT:D_DO-35_SOD27_P7.62mm_Horizontal" (at 186.69 128.27 0)
-      (effects (font (size 1.27 1.27)) hide)
-    )
-    (property "Datasheet" "https://assets.nexperia.com/documents/data-sheet/1N4148_1N4448.pdf" (at 186.69 128.27 0)
-      (effects (font (size 1.27 1.27)) hide)
-    )
-    (property "Sim.Device" "D" (at 186.69 128.27 0)
-      (effects (font (size 1.27 1.27)) hide)
-    )
-    (property "Sim.Pins" "1=K 2=A" (at 186.69 128.27 0)
-      (effects (font (size 1.27 1.27)) hide)
-    )
-    (pin "1")
-    (pin "2")
-    (instances
-      (project "stm_audio_board_V2"
-        (path "/6997cf63-2615-4e49-9471-e7da1b6bae71"
-          (reference "D4") (unit 1)
-        )
-        (path "/6997cf63-2615-4e49-9471-e7da1b6bae71/2eb2ee8f-ab98-4666-97f0-bfacb073bc88"
-          (reference "D4") (unit 1)
         )
       )
@@
       (effects (font (size 1.27 1.27)) (justify left))
     )
-    (property "Footprint" "Capacitor_THT:CP_Radial_D6.3mm_P2.50mm" (at 198.12 146.05 0)
-      (effects (font (size 1.27 1.27)) hide)
-    )
+    (property "Footprint" "Capacitor_SMD:CP_Elec_6.3x7.7" (at 198.12 146.05 0)
+      (effects (font (size 1.27 1.27)) hide)
+    )

Commit message: trace widening
Parts:
- C2: footprint Capacitor_THT:CP_Radial_D6.3mm_P2.50mm -> Capacitor_Tantalum_SMD:CP_EIA-7343-31_Kemet-D_Pad2.25x2.55mm_HandSolder
- C28, C29: footprint Capacitor_SMD:CP_Elec_6.3x7.7 -> Capacitor_Tantalum_SMD:CP_EIA-7343-31_Kemet-D_Pad2.25x2.55mm_HandSolder
Changed lines of the file:
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@@
       (effects (font (size 1.27 1.27)) (justify left))
     )
-    (property "Footprint" "Capacitor_SMD:CP_Elec_6.3x7.7" (at 175.26 147.32 0)
+    (property "Footprint" "Capacitor_Tantalum_SMD:CP_EIA-7343-31_Kemet-D_Pad2.25x2.55mm_HandSolder" (at 175.26 147.32 0)
       (effects (font (size 1.27 1.27)) hide)
     )
@@
       (effects (font (size 1.27 1.27)) (justify right))
     )
-    (property "Footprint" "Capacitor_THT:CP_Radial_D6.3mm_P2.50mm" (at 180.34 83.82 0)
+    (property "Footprint" "Capacitor_Tantalum_SMD:CP_EIA-7343-31_Kemet-D_Pad2.25x2.55mm_HandSolder" (at 180.34 83.82 0)
       (effects (font (size 1.27 1.27)) hide)
     )
@@
       (effects (font (size 1.27 1.27)) (justify left))
     )
-    (property "Footprint" "Capacitor_SMD:CP_Elec_6.3x7.7" (at 198.12 146.05 0)
+    (property "Footprint" "Capacitor_Tantalum_SMD:CP_EIA-7343-31_Kemet-D_Pad2.25x2.55mm_HandSolder" (at 198.12 146.05 0)
       (effects (font (size 1.27 1.27)) hide)
     )
@@
       (effects (font (size 1.27 1.27)) (justify left))
     )
-    (property "Footprint" "Capacitor_THT:CP_Radial_D6.3mm_P2.50mm" (at 171.45 90.17 0)
-      (effects (font (size 1.27 1.27)) hide)
-    )
+    (property "Footprint" "Capacitor_Tantalum_SMD:CP_EIA-7343-31_Kemet-D_Pad2.25x2.55mm_HandSolder" (at 171.45 90.17 0)
+      (effects (font (size 1.27 1.27)) hide)
+    )
