File: pcb/stm_audio_board_V2/Connectors.kicad_sch (KiCad schematic)
At the start: 11 parts, among them J1 Power conn, J2 STlink, J3 Audio_sig, J4 Conn_01x10_display, J6 Conn_01x03_pot_ext, J6 Conn_01x03_taptempo, J7 Conn_01x8_pots_internal

Commit message: pcb seems to be finished drc error: 0
Parts:
- removed J6: Conn_01x03_taptempo, Connector_PinHeader_2.54mm:PinHeader_1x03_P2.54mm_Vertical, symbol Connector_Generic:Conn_01x03
- added J4: Conn_01x01_taptempo, Connector_PinHeader_2.54mm:PinHeader_1x01_P2.54mm_Vertical, symbol Connector_Generic:Conn_01x01
Connections:
- net TAP_TEMPO_INPUT: now also J4.1 (Pin_1)
Changed lines of the file:
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@@
-    (stroke (width 0) (type default))
-  )
-  (wire (pts (xy 154.94 71.12) (xy 163.83 71.12))
     (stroke (width 0) (type default))
   )
@@
   )
   (wire (pts (xy 154.94 68.58) (xy 158.75 68.58))
-    (stroke (width 0) (type default))
-  )
-  (wire (pts (xy 154.94 66.04) (xy 163.83 66.04))
     (stroke (width 0) (type default))
   )
@@
         (path "/6997cf63-2615-4e49-9471-e7da1b6bae71/6424856c-1346-4018-a943-0d16008c9545"
           (reference "#PWR011") (unit 1)
-        )
-      )
-    )
-  )
-  (symbol (lib_id "Connector_Generic:Conn_01x03") (at 149.86 68.58 180) (unit 1)
-    (in_bom yes) (on_board yes) (dnp no)
-    (property "Reference" "J6" (at 146.05 67.31 0)
-      (effects (font (size 1.27 1.27)))
-    )
-    (property "Value" "Conn_01x03_taptempo" (at 137.16 69.85 0)
-      (effects (font (size 1.27 1.27)))
-    )
-    (property "Footprint" "Connector_PinHeader_2.54mm:PinHeader_1x03_P2.54mm_Vertical" (at 149.86 68.58 0)
-      (effects (font (size 1.27 1.27)) hide)
-    )
-    (property "Datasheet" "~" (at 149.86 68.58 0)
-      (effects (font (size 1.27 1.27)) hide)
-    )
-    (pin "1")
-    (pin "2")
-    (pin "3")
-    (instances
-      (project "stm_audio_board_V2"
-        (path "/6997cf63-2615-4e49-9471-e7da1b6bae71"
-          (reference "J6") (unit 1)
-        )
-        (path "/6997cf63-2615-4e49-9471-e7da1b6bae71/6424856c-1346-4018-a943-0d16008c9545"
-          (reference "J10") (unit 1)
         )
       )
@@
     )
   )
-  (symbol (lib_id "power:GND") (at 163.83 71.12 0) (unit 1)
-    (in_bom yes) (on_board yes) (dnp no) (fields_autoplaced)
-    (property "Reference" "#PWR050" (at 163.83 77.47 0)
-      (effects (font (size 1.27 1.27)) hide)
-    )
-    (property "Value" "GND" (at 163.83 76.2 0)
-      (effects (font (size 1.27 1.27)))
-    )
-    (property "Footprint" "" (at 163.83 71.12 0)
-      (effects (font (size 1.27 1.27)) hide)
-    )
-    (property "Datasheet" "" (at 163.83 71.12 0)
-      (effects (font (size 1.27 1.27)) hide)
-    )
-    (pin "1")
-    (instances
-      (project "stm_audio_board_V2"
-        (path "/6997cf63-2615-4e49-9471-e7da1b6bae71"
-          (reference "#PWR050") (unit 1)
-        )
-        (path "/6997cf63-2615-4e49-9471-e7da1b6bae71/6424856c-1346-4018-a943-0d16008c9545"
-          (reference "#PWR042") (unit 1)
-        )
-      )
-    )
-  )
   (symbol (lib_id "Mechanical:MountingHole_Pad") (at 102.87 58.42 90) (unit 1)
     (in_bom yes) (on_board yes) (dnp no) (fields_autoplaced)
@@
         (path "/6997cf63-2615-4e49-9471-e7da1b6bae71/6424856c-1346-4018-a943-0d16008c9545"
           (reference "#PWR064") (unit 1)
-        )
-      )
-    )
-  )
-  (symbol (lib_id "power:+3.3V") (at 163.83 66.04 0) (unit 1)
-    (in_bom yes) (on_board yes) (dnp no) (fields_autoplaced)
-    (property "Reference" "#PWR060" (at 163.83 69.85 0)
-      (effects (font (size 1.27 1.27)) hide)
-    )
-    (property "Value" "+3.3V" (at 163.83 62.23 0)
-      (effects (font (size 1.27 1.27)))
-    )
-    (property "Footprint" "" (at 163.83 66.04 0)
-      (effects (font (size 1.27 1.27)) hide)
-    )
-    (property "Datasheet" "" (at 163.83 66.04 0)
-      (effects (font (size 1.27 1.27)) hide)
-    )
-    (pin "1")
-    (instances
-      (project "stm_audio_board_V2"
-        (path "/6997cf63-2615-4e49-9471-e7da1b6bae71/6424856c-1346-4018-a943-0d16008c9545"
-          (reference "#PWR060") (unit 1)
         )
       )
@@
         )
       )
+    )
+  )
+  (symbol (lib_id "Connector_Generic:Conn_01x01") (at 149.86 68.58 180) (unit 1)
+    (in_bom yes) (on_board yes) (dnp no) (fields_autoplaced)
+    (property "Reference" "J4" (at 149.86 63.5 0)
+      (effects (font (size 1.27 1.27)))
+    )
+    (property "Value" "Conn_01x01_taptempo" (at 149.86 66.04 0)
+      (effects (font (size 1.27 1.27)))
+    )
+    (property "Footprint" "Connector_PinHeader_2.54mm:PinHeader_1x01_P2.54mm_Vertical" (at 149.86 68.58 0)
+      (effects (font (size 1.27 1.27)) hide)
+    )
+    (property "Datasheet" "~" (at 149.86 68.58 0)
+      (effects (font (size 1.27 1.27)) hide)
+    )
+    (pin "1")
+    (instances
+      (project "stm_audio_board_V2"
+        (path "/6997cf63-2615-4e49-9471-e7da1b6bae71/6424856c-1346-4018-a943-0d16008c9545"
+          (reference "J4") (unit 1)
+        )
+      )
