File: pcb/stm_audio_board_V2_1/MCU.kicad_sch (KiCad schematic)
At the start: 16 parts, among them SW1 SW_SPST, U1 STM32H747IGTx, Y2 X1E0000210132

Commit message: fixes in pcb
Connections:
- net +3.3V: no longer U1.102 (VDD12DSI), U1.108 (VDD12DSI), U1.113 (VDD), U1.126 (VDD), U1.13 (VDD), U1.136 (VDD), U1.152 (VDD), U1.160 (VDD), U1.176 (VDD), U1.25 (VDD), U1.44 (VDD), U1.48 (VDD), U1.65 (VDD), U1.7 (VDD), U1.71 (VDD), U1.8 (VBAT), U1.84 (VDD), U1.92 (VDD), U1.99 (VDD)
- net VDD_DSI: now reaches C13.1, U1.101 (VCAPDSI)
- net VDD_DSI: now also U1.102 (VDD12DSI), U1.108 (VDD12DSI)
- new net: U1.113 (VDD), U1.126 (VDD), U1.13 (VDD), U1.136 (VDD), U1.152 (VDD), U1.160 (VDD), U1.176 (VDD), U1.25 (VDD), U1.44 (VDD), U1.48 (VDD), U1.65 (VDD), U1.7 (VDD), U1.71 (VDD), U1.8 (VBAT), U1.84 (VDD), U1.92 (VDD), U1.99 (VDD)
Other:
- note added: "Crystal_OSC"
- note added: "LED"
- note added: "RESET"
- moved on the sheet: C16, C31, C37, D10, D11, R9, SW1, Y2
