File: pcb/stm_audio_board_V2_1/stm_audio_board_V2_1.kicad_sch (KiCad schematic)
At the start: 0 parts

Commit message: fixes in pcb
Other:
- added sheet Footswitch (Footswitch.kicad_sch)
Changed lines of the file:
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@@
+    )
+  )
+  (sheet (at 165.1 102.87) (size 36.83 26.67) (fields_autoplaced)
+    (stroke (width 0.1524) (type solid))
+    (fill (color 0 0 0 0.0000))
+    (property "Sheetname" "Footswitch" (at 165.1 102.1584 0)
+      (effects (font (size 1.27 1.27)) (justify left bottom))
+    )
+    (property "Sheetfile" "Footswitch.kicad_sch" (at 165.1 130.1246 0)
+      (effects (font (size 1.27 1.27)) (justify left top))
+    )
+    (instances
+      (project "stm_audio_board_V2_1"
+        (path "/6997cf63-2615-4e49-9471-e7da1b6bae71" (page "12"))
+      )
     )
   )
