File: pcb/stm_audio_board_V2_1/Output_stage.kicad_sch (KiCad schematic)
At the start: 29 parts, among them U2 OP275

Commit message: fixes in pcb
Connections:
- net GND: now also C41.1, R13.1; no longer C41.2, R13.2
- net at R17.2, U2.7: now also C41.2, R13.2; no longer C41.1, R13.1
- net at C41.1, R13.1: now also U2.6 (-); no longer U2.5 (+)
- net at C41.1, R13.1: now also U2.2 (-); no longer U2.3 (+)
- net at C41.2, R13.1: now also U2.3 (+); no longer U2.2 (-)
- net at C41.2, R13.1: now also U2.5 (+); no longer U2.6 (-)
Other:
- moved on the sheet: U2A, U2B

Commit message: audo_board v2_1 output stage is reworked
Connections:
- net at C41.1, U2.6 (-): now also R13.2; no longer R13.1
- net at C41.2, R13.1, R13.2: now also R13.1; no longer R13.2
- net DAC1L renamed DAC1N
- net DAC1R renamed DAC1P
- net DAC2L renamed DAC2P
- net DAC2R renamed DAC2N
Other:
- moved on the sheet: R13
Changed lines of the file:
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@@
     (stroke (width 0) (type default))
   )
-  (wire (pts (xy 78.74 58.42) (xy 80.01 58.42))
+  (wire (pts (xy 69.85 58.42) (xy 80.01 58.42))
     (stroke (width 0) (type default))
   )
@@
     (stroke (width 0) (type default))
   )
-  (wire (pts (xy 78.74 82.55) (xy 80.01 82.55))
+  (wire (pts (xy 69.85 82.55) (xy 80.01 82.55))
     (stroke (width 0) (type default))
   )
@@
     )
   )
+  (global_label "DAC2P" (shape input) (at 78.74 146.05 180) (fields_autoplaced)
+    (effects (font (size 1.27 1.27)) (justify right))
+    (property "Intersheetrefs" "${INTERSHEET_REFS}" (at 69.7261 146.05 0)
+      (effects (font (size 1.27 1.27)) (justify right) hide)
+    )
+  )
   (global_label "GUITAR_OUT_R" (shape input) (at 175.26 133.35 0) (fields_autoplaced)
     (effects (font (size 1.27 1.27)) (justify left))
@@
     )
   )
-  (global_label "DAC1R" (shape input) (at 78.74 58.42 180) (fields_autoplaced)
-    (effects (font (size 1.27 1.27)) (justify right))
-    (property "Intersheetrefs" "${INTERSHEET_REFS}" (at 69.7261 58.42 0)
-      (effects (font (size 1.27 1.27)) (justify right) hide)
-    )
-  )
-  (global_label "DAC1L" (shape input) (at 78.74 82.55 180) (fields_autoplaced)
-    (effects (font (size 1.27 1.27)) (justify right))
-    (property "Intersheetrefs" "${INTERSHEET_REFS}" (at 69.968 82.55 0)
-      (effects (font (size 1.27 1.27)) (justify right) hide)
-    )
-  )
-  (global_label "DAC2R" (shape input) (at 78.74 121.92 180) (fields_autoplaced)
-    (effects (font (size 1.27 1.27)) (justify right))
-    (property "Intersheetrefs" "${INTERSHEET_REFS}" (at 69.7261 121.92 0)
-      (effects (font (size 1.27 1.27)) (justify right) hide)
-    )
-  )
-  (global_label "DAC2L" (shape input) (at 78.74 146.05 180) (fields_autoplaced)
-    (effects (font (size 1.27 1.27)) (justify right))
-    (property "Intersheetrefs" "${INTERSHEET_REFS}" (at 69.968 146.05 0)
+  (global_label "DAC2N" (shape input) (at 78.74 121.92 180) (fields_autoplaced)
+    (effects (font (size 1.27 1.27)) (justify right))
+    (property "Intersheetrefs" "${INTERSHEET_REFS}" (at 69.6656 121.92 0)
+      (effects (font (size 1.27 1.27)) (justify right) hide)
+    )
+  )
+  (global_label "DAC1P" (shape input) (at 69.85 58.42 180) (fields_autoplaced)
+    (effects (font (size 1.27 1.27)) (justify right))
+    (property "Intersheetrefs" "${INTERSHEET_REFS}" (at 60.8361 58.42 0)
+      (effects (font (size 1.27 1.27)) (justify right) hide)
+    )
+  )
+  (global_label "DAC1N" (shape input) (at 69.85 82.55 180) (fields_autoplaced)
+    (effects (font (size 1.27 1.27)) (justify right))
+    (property "Intersheetrefs" "${INTERSHEET_REFS}" (at 60.7756 82.55 0)
       (effects (font (size 1.27 1.27)) (justify right) hide)
     )
@@
     )
   )
-  (symbol (lib_id "Device:R") (at 105.41 58.42 270) (unit 1)
-    (in_bom yes) (on_board yes) (dnp no) (fields_autoplaced)
+  (symbol (lib_id "Device:R") (at 105.41 58.42 90) (mirror x) (unit 1)
+    (in_bom yes) (on_board yes) (dnp no)
     (property "Reference" "R13" (at 105.41 53.34 90)
       (effects (font (size 1.27 1.27)))
