File: pcb/stm_audio_board_V2_1/stm_audio_board_V2_1.kicad_pcb (KiCad board)
At the start: 4 copper layers, 66.1 x 71 mm, 152 parts, among them J1 Power conn, J2 STlink, J3 Audio_sig, J4 Conn_01x01_taptempo, J5 Conn_01x10_display, J6 Conn_01x03_pot_ext, J7 Conn_01x8_pots_internal, SW1 SW_SPST, U1 STM32H747IGTx, U2 OP275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

Commit message: audo_board v2_1 output stage is reworked
Parts:
- removed C65, C66: 10p, Capacitor_SMD:C_0603_1608Metric_Pad1.08x0.95mm_HandSolder
- removed D7: LED, LED_SMD:LED_SK6805_PLCC4_2.4x2.7mm_P1.3mm
- removed R28: 10k, Resistor_SMD:R_0805_2012Metric_Pad1.20x1.40mm_HandSolder
- removed Y1: Crystal_GND24, Crystal:Crystal_SMD_5032-4Pin_5.0x3.2mm
- C19: value 220p -> 10p
- C20: value 120p -> 10p
- C67: value 5.6nF -> 39nF
- C68: value 390pF -> 2.2nF
- R10: value 562 -> 3.32k
- moved C45 8.59 mm to (207.4, 110.8), turned to 180 degrees
- moved C38 8.20 mm to (208.2, 106.3), turned to 90 degrees
- moved C44 6.77 mm to (203.6, 108.1), turned to 180 degrees
- moved R22 5.41 mm to (199.7, 108.1)
- moved C41 5.08 mm to (201.9, 104.3)
- moved R15 5.02 mm to (205.0, 101.6)
- moved R16 4.97 mm to (202.6, 101.6)
- moved C40 4.90 mm to (205.6, 104.3)
- moved R21 4.78 mm to (207.3, 108.1), turned to 0 degrees
- moved R19 4.77 mm to (205.8, 106.1), turned to 180 degrees
- moved R20 4.69 mm to (201.8, 106.1)
- moved C89 4.21 mm to (200.6, 106.1), turned to -90 degrees
- moved R13 2.60 mm to (202.9, 100.9), turned to 0 degrees
- moved C39 2.23 mm to (204.6, 102.8)
- moved R14 1.38 mm to (208.2, 102.8)
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Connections:
- net DAC1L renamed DAC1N
- net DAC1R renamed DAC1P
- C2 pad 1: Net-(U1-VCAPDSI) -> /MCU/VDD_DSI
- C38 pad 1: Net-(C38-Pad1) -> GND
- C38 pad 2: Net-(U2B--) -> Net-(U2B-+)
- C39 pad 1: Net-(U2B-+) -> Net-(U2B--)
- C39 pad 2: GND -> Net-(C39-Pad2)
- C44 pad 1: Net-(U2A-+) -> Net-(U2A--)
- C45 pad 2: Net-(U2A--) -> Net-(U2A-+)
- C68 pad 1: GND -> +3.3VA
- R10 pad 2: GND -> +3.3VA
- R13 pad 1: Net-(U2B-+) -> Net-(C22-Pad2)
- R13 pad 2: Net-(C22-Pad2) -> Net-(U2B--)
- R14 pad 1: Net-(U2B--) -> Net-(U2B-+)
- R15 pad 1: DAC2R -> DAC2N
- R16 pad 1: DAC2L -> DAC2P
- R17 pad 2: Net-(C38-Pad1) -> Net-(C39-Pad2)
- R21 pad 1: Net-(U2A-+) -> Net-(U2A--)
- R22 pad 1: Net-(U2A--) -> Net-(U2A-+)
- R31 pad 2: GND -> Net-(C39-Pad2)
- R32 pad 1: Net-(C38-Pad1) -> GND
- U1 pad 101: Net-(U1-VCAPDSI) -> /MCU/VDD_DSI
- U1 pad 102: +3.3V -> /MCU/VDD_DSI
- U1 pad 108: +3.3V -> /MCU/VDD_DSI
- U1 pad 113: +3.3V -> Net-(U1-VBAT)
- U1 pad 126: +3.3V -> Net-(U1-VBAT)
- U1 pad 13: +3.3V -> Net-(U1-VBAT)
- U1 pad 136: +3.3V -> Net-(U1-VBAT)
- U1 pad 152: +3.3V -> Net-(U1-VBAT)
- U1 pad 160: +3.3V -> Net-(U1-VBAT)
- U1 pad 176: +3.3V -> Net-(U1-VBAT)
- U1 pad 25: +3.3V -> Net-(U1-VBAT)
- U1 pad 44: +3.3V -> Net-(U1-VBAT)
- U1 pad 48: +3.3V -> Net-(U1-VBAT)
- U1 pad 65: +3.3V -> Net-(U1-VBAT)
- U1 pad 7: +3.3V -> Net-(U1-VBAT)
- U1 pad 71: +3.3V -> Net-(U1-VBAT)
- U1 pad 8: +3.3V -> Net-(U1-VBAT)
- U1 pad 84: +3.3V -> Net-(U1-VBAT)
- U1 pad 92: +3.3V -> Net-(U1-VBAT)
- U1 pad 99: +3.3V -> Net-(U1-VBAT)
- U11 pad 42: DAC2R -> DAC2P
- U11 pad 43: DAC2L -> DAC2N
- U11 pad 5: GND -> +3.3VA
- U2 pad 7: Net-(C38-Pad1) -> Net-(C39-Pad2)
Routing:
- net GND: track 221.9 -> 194.4 mm, vias 331 -> 302
- net Net-(C39-Pad2): track 0.00 -> 16.2 mm
- net -9V: track 47.6 -> 63.2 mm
- net +9V: track 88.4 -> 103.6 mm, vias 2 -> 1
- net DAC2P: track 0.00 -> 11.9 mm, vias 0 -> 1
- net DAC2N: track 0.00 -> 11.4 mm, vias 0 -> 1
- net AD1939_MCLKI: track 11.1 -> 0.00 mm, vias 1 -> 0
- net Net-(C44-Pad2): track 19.7 -> 9.65 mm, vias 2 -> 1
- net DAC2L: track 9.19 -> 0.00 mm, vias 1 -> 0
- net Net-(U2A--): track 13.7 -> 4.81 mm
- net AD1939_MCLKO: track 8.74 -> 0.00 mm, vias 1 -> 0
- net +3.3VA: track 73.5 -> 81.1 mm
- net DAC2R: track 6.07 -> 0.00 mm, vias 1 -> 0
- net +3.3V: track 318.6 -> 314.7 mm
- net Net-(U1-VBAT): track 0.00 -> 3.92 mm
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Other:
- board text added: "STM_AUDIO_BOARD_V2/1"
- board text removed: "STM_AUDIO_BOARD_V2"
